Commit message: \#13 Updated urdf

File: c3pzero_description/src/description/c3pzero_description.urdf (robot description, URDF)
Before this commit: robot sam_bot, 7 links, 6 joints
Links:
- removed link camera_depth_frame
- removed link camera_link
- removed link imu_link
Joints:
- removed joint camera_depth_joint
- removed joint camera_joint
- removed joint imu_joint
- joint caster_joint: origin xyz=${caster_xoff} 0.0 ${-(base_height/2)} rpy=0 0 0 -> xyz=${-caster_xoff} 0.0 ${-(base_height/2)} rpy=0 0 0
- joint lidar_joint: origin xyz=0 0 0.12 rpy=0 0 0 -> xyz=0.20 0 0.17 rpy=0 0 0
