Commit message: add robot mesh files

File: c3pzero_description/urdf/c3pzero_description.urdf (robot description, URDF)
Before this commit: robot c3pzero, 4 links, 3 joints
Links:
- removed link front_caster
- added link lr_caster; collision sphere radius=${(wheel_radius-(base_height/2))}; visual sphere radius=${(wheel_radius-(base_height/2))}
- added link rr_caster; collision sphere radius=${(wheel_radius-(base_height/2))}; visual sphere radius=${(wheel_radius-(base_height/2))}
- link base_link: geometry collision box size=${base_length} ${base_width} ${base_height}; visual mesh filename=file://$(find c3pzero_description)/urdf/meshes/c300_base_li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
Joints:
- removed joint caster_joint
- added joint lr_caster_joint: type fixed, parent base_link, child lr_caster, origin xyz=${-caster_xoff} -0.193 ${-(base_height/2)} rpy=0 0 0
- added joint rr_caster_joint: type fixed, parent base_link, child rr_caster, origin xyz=${-caster_xoff} 0.193 ${-(base_height/2)} rpy=0 0 0
- joint base_joint: origin xyz=0.0 0.0 ${-(wheel_radius+wheel_zoff)} rpy=0 0 0 -> xyz=0.0 0.0 ${-wheel_radius} rpy=0 0 0
- joint lidar_joint: origin xyz=0.20 0 0.17 rpy=0 0 0 -> xyz=0 0 0.19 rpy=0 0 0
